File: hoperf-rfm9x-lora-breakout.sch (EAGLE design)
At the start: 6 parts, among them U1 HopeRF-RFM9x

Commit message: rfm9x lora breakout v1.1
Parts:
- added LOGO1: OSHW-LOGOS, SparkFun-Aesthetics:OSHW-LOGOS
- added U$3: LORA_LOGO, #afb-Aesthetics:LORA_LOGO
Other:
- note added: "github.com/altro-id"
- moved on the sheet: ANT, C1, JP1, JP2, U1, UFL/SMA
Changed lines of the file:
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@@
 <part name="ANT" library="microbuilder" deviceset="HEADER-1X1" device="ROUND"/>
 <part name="UFL/SMA" library="#afb-Connectors" deviceset="MICROBUILDER_SMACONNECTOR" device="_EDGE_UFL"/>
-<part name="FRAME1" library="#afb-Aesthetics" deviceset="A5L-LOC" device=""/>
+<part name="LOGO1" library="SparkFun-Aesthetics" deviceset="OSHW-LOGO" device="S"/>
+<part name="U$3" library="#afb-Aesthetics" deviceset="LORA_LOGO" device=""/>
 </parts>
 <sheets>
 <sheet>
 <plain>
-<text x="88.9" y="15.24" size="1.9304" layer="94" font="vector" ratio="14">HopeRF RFM95/6/7/8 LoRa(TM)
+<text x="30.48" y="10.16" size="1.9304" layer="94" font="vector" ratio="14">HopeRF RFM95/6/7/8 LoRa(TM)
 Module Breakout Board</text>
+<text x="30.48" y="5.08" size="1.778" layer="95" font="vector">github.com/altro-id</text>
 </plain>
 <instances>
-<instance part="U1" gate="G$1" x="86.36" y="78.74"/>
-<instance part="JP1" gate="A" x="53.34" y="78.74" rot="MR0"/>
-<instance part="C1" gate="G$1" x="127" y="76.2"/>
-<instance part="U$1" gate="G$1" x="127" y="68.58"/>
-<instance part="U$19" gate="G$1" x="109.22" y="45.72" rot="MR0"/>
-<instance part="U$2" gate="G$1" x="93.98" y="45.72" rot="MR0"/>
-<instance part="JP2" gate="A" x="119.38" y="81.28"/>
-<instance part="ANT" gate="G$1" x="99.06" y="66.04" rot="R180"/>
-<instance part="UFL/SMA" gate="G$1" x="101.6" y="53.34" rot="R270"/>
-<instance part="FRAME1" gate="G$1" x="0" y="0"/>
+<instance part="U1" gate="G$1" x="45.72" y="66.04"/>
+<instance part="JP1" gate="A" x="12.7" y="66.04" rot="MR0"/>
+<instance part="C1" gate="G$1" x="86.36" y="63.5"/>
+<instance part="U$1" gate="G$1" x="86.36" y="55.88"/>
+<instance part="U$19" gate="G$1" x="68.58" y="33.02" rot="MR0"/>
+<instance part="U$2" gate="G$1" x="53.34" y="33.02" rot="MR0"/>
+<instance part="JP2" gate="A" x="78.74" y="68.58"/>
+<instance part="ANT" gate="G$1" x="58.42" y="53.34" rot="R180"/>
+<instance part="UFL/SMA" gate="G$1" x="60.96" y="40.64" rot="R270"/>
+<instance part="LOGO1" gate="G$1" x="12.7" y="17.78"/>
+<instance part="U$3" gate="G$1" x="2.54" y="5.08"/>
 </instances>
 <busses>
@@
 <pinref part="U1" gate="G$1" pin="MOSI"/>
 <pinref part="JP1" gate="A" pin="3"/>
-<wire x1="55.88" y1="83.82" x2="71.12" y2="83.82" width="0.1524" layer="91"/>
+<wire x1="15.24" y1="71.12" x2="30.48" y2="71.12" width="0.1524" layer="91"/>
 </segment>
 </net>
@@
 <pinref part="U1" gate="G$1" pin="SCK"/>
 <pinref part="JP1" gate="A" pin="4"/>
-<wire x1="55.88" y1="81.28" x2="71.12" y2="81.28" width="0.1524" layer="91"/>
+<wire x1="15.24" y1="68.58" x2="30.48" y2="68.58" width="0.1524" layer="91"/>
 </segment>
 </net>
@@
 <pinref part="U1" gate="G$1" pin="NSS"/>
 <pinref part="JP1" gate="A" pin="5"/>
-<wire x1="55.88" y1="78.74" x2="71.12" y2="78.74" width="0.1524" layer="91"/>
+<wire x1="15.24" y1="66.04" x2="30.48" y2="66.04" width="0.1524" layer="91"/>
 </segment>
 </net>
@@
 <pinref part="U1" gate="G$1" pin="RESET"/>
 <pinref part="JP1" gate="A" pin="6"/>
-<wire x1="55.88" y1="76.2" x2="71.12" y2="76.2" width="0.1524" layer="91"/>
+<wire x1="15.24" y1="63.5" x2="30.48" y2="63.5" width="0.1524" layer="91"/>
 </segment>
 </net>
@@
 <segment>
 <pinref part="U$19" gate="G$1" pin="GND"/>
-<junction x="109.22" y="50.8"/>
-<junction x="109.22" y="50.8"/>
-<wire x1="109.22" y1="50.8" x2="109.22" y2="55.88" width="0.1524" layer="91"/>
+<junction x="68.58" y="38.1"/>
+<junction x="68.58" y="38.1"/>
+<wire x1="68.58" y1="38.1" x2="68.58" y2="43.18" width="0.1524" layer="91"/>
 <pinref part="U1" gate="G$1" pin="GND@1"/>
-<wire x1="109.22" y1="55.88" x2="109.22" y2="73.66" width="0.1524" layer="91"/>
-<wire x1="101.6" y1="73.66" x2="109.22" y2="73.66" width="0.1524" layer="91"/>
-<junction x="109.22" y="50.8"/>
-<wire x1="109.22" y1="50.8" x2="109.22" y2="48.26" width="0.1524" layer="91"/>
+<wire x1="68.58" y1="43.18" x2="68.58" y2="60.96" width="0.1524" layer="91"/>
+<wire x1="60.96" y1="60.96" x2="68.58" y2="60.96" width="0.1524" layer="91"/>
+<junction x="68.58" y="38.1"/>
+<wire x1="68.58" y1="38.1" x2="68.58" y2="35.56" width="0.1524" layer="91"/>
 <pinref part="UFL/SMA" gate="G$1" pin="GND1"/>
-<junction x="109.22" y="55.88"/>
+<junction x="68.58" y="43.18"/>
 <pinref part="UFL/SMA" gate="G$1" pin="GND2"/>
 </segment>
@@
 <pinref part="U1" gate="G$1" pin="GND@2"/>
 <pinref part="JP1" gate="A" pin="1"/>
-<wire x1="55.88" y1="88.9" x2="71.12" y2="88.9" width="0.1524" layer="91"/>
+<wire x1="15.24" y1="76.2" x2="30.48" y2="76.2" width="0.1524" layer="91"/>
 </segment>
 <segment>
 <pinref part="U1" gate="G$1" pin="GND@3"/>
 <pinref part="JP1" gate="A" pin="8"/>
-<wire x1="55.88" y1="71.12" x2="71.12" y2="71.12" width="0.1524" layer="91"/>
+<wire x1="15.24" y1="58.42" x2="30.48" y2="58.42" width="0.1524" layer="91"/>
 </segment>
 <segment>
 <pinref part="U$2" gate="G$1" pin="GND"/>
-<wire x1="93.98" y1="48.26" x2="93.98" y2="50.8" width="0.1524" layer="91"/>
+<wire x1="53.34" y1="35.56" x2="53.34" y2="38.1" width="0.1524" layer="91"/>
 <pinref part="UFL/SMA" gate="G$1" pin="GND3"/>
 <pinref part="UFL/SMA" gate="G$1" pin="GND4"/>
-<wire x1="93.98" y1="50.8" x2="93.98" y2="55.88" width="0.1524" layer="91"/>
-<junction x="93.98" y="50.8"/>
+<wire x1="53.34" y1="38.1" x2="53.34" y2="43.18" width="0.1524" layer="91"/>
+<junction x="53.34" y="38.1"/>
 </segment>
 </net>
@@
 <pinref part="U1" gate="G$1" pin="MISO"/>
 <pinref part="JP1" gate="A" pin="2"/>
-<wire x1="55.88" y1="86.36" x2="71.12" y2="86.36" width="0.1524" layer="91"/>
+<wire x1="15.24" y1="73.66" x2="30.48" y2="73.66" width="0.1524" layer="91"/>
 </segment>
 </net>
@@
 <pinref part="U1" gate="G$1" pin="DIO5"/>
 <pinref part="JP1" gate="A" pin="7"/>
-<wire x1="55.88" y1="73.66" x2="71.12" y2="73.66" width="0.1524" layer="91"/>
+<wire x1="15.24" y1="60.96" x2="30.48" y2="60.96" width="0.1524" layer="91"/>
 </segment>
 </net>
@@
 <segment>
 <pinref part="U1" gate="G$1" pin="DIO2"/>
-<wire x1="116.84" y1="88.9" x2="101.6" y2="88.9" width="0.1524" layer="91"/>
+<wire x1="76.2" y1="76.2" x2="60.96" y2="76.2" width="0.1524" layer="91"/>
 <pinref part="JP2" gate="A" pin="1"/>
 </segment>
@@
 <segment>
 <pinref part="U1" gate="G$1" pin="DIO1"/>
-<wire x1="116.84" y1="86.36" x2="101.6" y2="86.36" width="0.1524" layer="91"/>
+<wire x1="76.2" y1="73.66" x2="60.96" y2="73.66" width="0.1524" layer="91"/>
 <pinref part="JP2" gate="A" pin="2"/>
 </segment>
@@
 <segment>
 <pinref part="U1" gate="G$1" pin="DIO0"/>
-<wire x1="116.84" y1="83.82" x2="101.6" y2="83.82" width="0.1524" layer="91"/>
+<wire x1="76.2" y1="71.12" x2="60.96" y2="71.12" width="0.1524" layer="91"/>
 <pinref part="JP2" gate="A" pin="3"/>
 </segment>
@@
 <segment>
 <pinref part="U1" gate="G$1" pin="3.3V"/>
-<wire x1="127" y1="81.28" x2="116.84" y2="81.28" width="0.1524" layer="91"/>
+<wire x1="86.36" y1="68.58" x2="76.2" y2="68.58" width="0.1524" layer="91"/>
 <pinref part="C1" gate="G$1" pin="1"/>
-<wire x1="116.84" y1="81.28" x2="101.6" y2="81.28" width="0.1524" layer="91"/>
-<wire x1="127" y1="81.28" x2="127" y2="78.74" width="0.1524" layer="91"/>
-<junction x="116.84" y="81.28"/>
+<wire x1="76.2" y1="68.58" x2="60.96" y2="68.58" width="0.1524" layer="91"/>
+<wire x1="86.36" y1="68.58" x2="86.36" y2="66.04" width="0.1524" layer="91"/>
+<junction x="76.2" y="68.58"/>
 <pinref part="JP2" gate="A" pin="4"/>
 </segment>
@@
 <segment>
 <pinref part="U1" gate="G$1" pin="DIO4"/>
-<wire x1="116.84" y1="78.74" x2="101.6" y2="78.74" width="0.1524" layer="91"/>
+<wire x1="76.2" y1="66.04" x2="60.96" y2="66.04" width="0.1524" layer="91"/>
 <pinref part="JP2" gate="A" pin="5"/>
 </segment>
@@
 <segment>
 <pinref part="U1" gate="G$1" pin="DIO3"/>
-<wire x1="116.84" y1="76.2" x2="101.6" y2="76.2" width="0.1524" layer="91"/>
+<wire x1="76.2" y1="63.5" x2="60.96" y2="63.5" width="0.1524" layer="91"/>
 <pinref part="JP2" gate="A" pin="6"/>
 </segment>
@@
 <segment>
 <pinref part="U1" gate="G$1" pin="ANT"/>
-<wire x1="101.6" y1="71.12" x2="101.6" y2="66.04" width="0.1524" layer="91"/>
+<wire x1="60.96" y1="58.42" x2="60.96" y2="53.34" width="0.1524" layer="91"/>
 <pinref part="ANT" gate="G$1" pin="1"/>
-<wire x1="101.6" y1="66.04" x2="101.6" y2="60.96" width="0.1524" layer="91"/>
-<junction x="101.6" y="66.04"/>
+<wire x1="60.96" y1="53.34" x2="60.96" y2="48.26" width="0.1524" layer="91"/>
+<junction x="60.96" y="53.34"/>
 <pinref part="UFL/SMA" gate="G$1" pin="ANT"/>
 </segment>
